Commit message: Add MoveIt packages for all robots
Added MoveIt packages for TX60, TX60L, TX90L, TX90XL

File: staubli_tx60_support/urdf/tx60_macro.xacro (robot description, xacro)
@@ -167,5 +167,5 @@
       (1) effort limit = 126 Nm if floor mounted
       (2) effort limit = 65 Nm if wall mounted -->
-      <limit lower="${radians(-180)}" upper="${radians(180)}" effort="126.0" velocity="${radians(435)}" />
+      <limit lower="${radians(-180)}" upper="${radians(180)}" effort="126.0" velocity="${radians(287)}" />
       <dynamics damping="0.0" friction="0.0"/>
     </joint>
@@ -175,5 +175,5 @@
       <child link="${prefix}link_2"/>
       <axis xyz="0 1 0"/>
-      <limit lower="${radians(-127.5)}" upper="${radians(127.5)}" effort="71.0" velocity="${radians(410)}" />
+      <limit lower="${radians(-127.5)}" upper="${radians(127.5)}" effort="71.0" velocity="${radians(287)}" />
       <dynamics damping="0.0" friction="0.0"/>
     </joint>
@@ -183,5 +183,5 @@
       <child link="${prefix}link_3"/>
       <axis xyz="0 1 0"/>
-      <limit lower="${radians(-142.5)}" upper="${radians(142.5)}" effort="38.0" velocity="${radians(540)}" />
+      <limit lower="${radians(-142.5)}" upper="${radians(142.5)}" effort="38.0" velocity="${radians(431)}" />
       <dynamics damping="0.0" friction="0.0"/>
     </joint>
@@ -191,5 +191,5 @@
       <child link="${prefix}link_4"/>
       <axis xyz="0 0 1"/>
-      <limit lower="${radians(-270.0)}" upper="${radians(270.0)}" effort="7.0" velocity="${radians(995)}" />
+      <limit lower="${radians(-270.0)}" upper="${radians(270.0)}" effort="7.0" velocity="${radians(410)}" />
       <dynamics damping="0.0" friction="0.0"/>
     </joint>
@@ -199,5 +199,5 @@
       <child link="${prefix}link_5"/>
       <axis xyz="0 1 0"/>
-      <limit lower="${radians(-122.5)}" upper="${radians(132.5)}" effort="8.0" velocity="${radians(1065)}" />
+      <limit lower="${radians(-122.5)}" upper="${radians(132.5)}" effort="8.0" velocity="${radians(320)}" />
       <dynamics damping="0.0" friction="0.0"/>
     </joint>
@@ -207,5 +207,5 @@
       <child link="${prefix}link_6"/>
       <axis xyz="0 0 1"/>
-      <limit lower="${radians(-270.0)}" upper="${radians(270.0)}" effort="2.0" velocity="${radians(1445)}" />
+      <limit lower="${radians(-270.0)}" upper="${radians(270.0)}" effort="2.0" velocity="${radians(700)}" />
       <dynamics damping="0.0" friction="0.0"/>
     </joint>

File: staubli_tx60_support/urdf/tx60l_macro.xacro (robot description, xacro)
@@ -167,5 +167,5 @@
       (1) effort limit = 126 Nm if floor mounted
       (2) effort limit = 40 Nm if wall mounted -->
-      <limit lower="${radians(-180)}" upper="${radians(180)}" effort="126.0" velocity="${radians(435)}" />
+      <limit lower="${radians(-180)}" upper="${radians(180)}" effort="126.0" velocity="${radians(287)}" />
       <dynamics damping="0.0" friction="0.0"/>
     </joint>
@@ -175,5 +175,5 @@
       <child link="${prefix}link_2"/>
       <axis xyz="0 1 0"/>
-      <limit lower="${radians(-127.5)}" upper="${radians(127.5)}" effort="47.0" velocity="${radians(385)}" />
+      <limit lower="${radians(-127.5)}" upper="${radians(127.5)}" effort="47.0" velocity="${radians(287)}" />
       <dynamics damping="0.0" friction="0.0"/>
     </joint>
@@ -183,5 +183,5 @@
       <child link="${prefix}link_3"/>
       <axis xyz="0 1 0"/>
-      <limit lower="${radians(-152.5)}" upper="${radians(152.5)}" effort="32.0" velocity="${radians(500)}" />
+      <limit lower="${radians(-152.5)}" upper="${radians(152.5)}" effort="32.0" velocity="${radians(431)}" />
       <dynamics damping="0.0" friction="0.0"/>
     </joint>
@@ -191,5 +191,5 @@
       <child link="${prefix}link_4"/>
       <axis xyz="0 0 1"/>
-      <limit lower="${radians(-270.0)}" upper="${radians(270.0)}" effort="7.0" velocity="${radians(995)}" />
+      <limit lower="${radians(-270.0)}" upper="${radians(270.0)}" effort="7.0" velocity="${radians(410)}" />
       <dynamics damping="0.0" friction="0.0"/>
     </joint>
@@ -199,5 +199,5 @@
       <child link="${prefix}link_5"/>
       <axis xyz="0 1 0"/>
-      <limit lower="${radians(-122.5)}" upper="${radians(132.5)}" effort="8.0" velocity="${radians(1065)}" />
+      <limit lower="${radians(-122.5)}" upper="${radians(132.5)}" effort="8.0" velocity="${radians(320)}" />
       <dynamics damping="0.0" friction="0.0"/>
     </joint>
@@ -207,5 +207,5 @@
       <child link="${prefix}link_6"/>
       <axis xyz="0 0 1"/>
-      <limit lower="${radians(-270.0)}" upper="${radians(270.0)}" effort="2.0" velocity="${radians(1445)}" />
+      <limit lower="${radians(-270.0)}" upper="${radians(270.0)}" effort="2.0" velocity="${radians(700)}" />
       <dynamics damping="0.0" friction="0.0"/>
     </joint>

File: staubli_tx90_support/urdf/tx90_macro.xacro (robot description, xacro)
@@ -167,5 +167,5 @@
       (1) effort limit = 318 Nm if floor mounted
       (2) effort limit = 111 Nm if wall mounted -->
-      <limit lower="${radians(-180)}" upper="${radians(180)}" effort="318.0" velocity="${radians(400)}" />
+      <limit lower="${radians(-180)}" upper="${radians(180)}" effort="318.0" velocity="${radians(250)}" />
       <dynamics damping="0.0" friction="0.0"/>
     </joint>
@@ -175,5 +175,5 @@
       <child link="${prefix}link_2"/>
       <axis xyz="0 1 0"/>
-      <limit lower="${radians(-130)}" upper="${radians(147.5)}" effort="166.0" velocity="${radians(400)}" />
+      <limit lower="${radians(-130)}" upper="${radians(147.5)}" effort="166.0" velocity="${radians(200)}" />
       <dynamics damping="0.0" friction="0.0"/>
     </joint>
@@ -183,5 +183,5 @@
       <child link="${prefix}link_3"/>
       <axis xyz="0 1 0"/>
-      <limit lower="${radians(-145)}" upper="${radians(145)}" effort="76.0" velocity="${radians(430)}" />
+      <limit lower="${radians(-145)}" upper="${radians(145)}" effort="76.0" velocity="${radians(300)}" />
       <dynamics damping="0.0" friction="0.0"/>
     </joint>
@@ -191,5 +191,5 @@
       <child link="${prefix}link_4"/>
       <axis xyz="0 0 1"/>
-      <limit lower="${radians(-270)}" upper="${radians(270)}" effort="34.0" velocity="${radians(540)}" />
+      <limit lower="${radians(-270)}" upper="${radians(270)}" effort="34.0" velocity="${radians(430)}" />
       <dynamics damping="0.0" friction="0.0"/>
     </joint>
@@ -199,5 +199,5 @@
       <child link="${prefix}link_5"/>
       <axis xyz="0 1 0"/>
-      <limit lower="${radians(-115)}" upper="${radians(140)}" effort="29.0" velocity="${radians(475)}" />
+      <limit lower="${radians(-115)}" upper="${radians(140)}" effort="29.0" velocity="${radians(350)}" />
       <dynamics damping="0.0" friction="0.0"/>
     </joint>
@@ -207,5 +207,5 @@
       <child link="${prefix}link_6"/>
       <axis xyz="0 0 1"/>
-      <limit lower="${radians(-270)}" upper="${radians(270)}" effort="11.0" velocity="${radians(760)}" />
+      <limit lower="${radians(-270)}" upper="${radians(270)}" effort="11.0" velocity="${radians(600)}" />
       <dynamics damping="0.0" friction="0.0"/>
     </joint>

File: staubli_tx90_support/urdf/tx90l_macro.xacro (robot description, xacro)
@@ -167,5 +167,5 @@
       (1) effort limit = 318 Nm if floor mounted
       (2) effort limit = 111 Nm if wall mounted -->
-      <limit lower="${radians(-180)}" upper="${radians(180)}" effort="318.0" velocity="${radians(400)}" />
+      <limit lower="${radians(-180)}" upper="${radians(180)}" effort="318.0" velocity="${radians(215)}" />
       <dynamics damping="0.0" friction="0.0"/>
     </joint>
@@ -175,5 +175,5 @@
       <child link="${prefix}link_2"/>
       <axis xyz="0 1 0"/>
-      <limit lower="${radians(-130)}" upper="${radians(147.5)}" effort="130.0" velocity="${radians(390)}" />
+      <limit lower="${radians(-130)}" upper="${radians(147.5)}" effort="130.0" velocity="${radians(170)}" />
       <dynamics damping="0.0" friction="0.0"/>
     </joint>
@@ -183,5 +183,5 @@
       <child link="${prefix}link_3"/>
       <axis xyz="0 1 0"/>
-      <limit lower="${radians(-145)}" upper="${radians(145)}" effort="65.0" velocity="${radians(420)}" />
+      <limit lower="${radians(-145)}" upper="${radians(145)}" effort="65.0" velocity="${radians(255)}" />
       <dynamics damping="0.0" friction="0.0"/>
     </joint>
@@ -191,5 +191,5 @@
       <child link="${prefix}link_4"/>
       <axis xyz="0 0 1"/>
-      <limit lower="${radians(-270)}" upper="${radians(270)}" effort="34.0" velocity="${radians(540)}" />
+      <limit lower="${radians(-270)}" upper="${radians(270)}" effort="34.0" velocity="${radians(430)}" />
       <dynamics damping="0.0" friction="0.0"/>
     </joint>
@@ -199,5 +199,5 @@
       <child link="${prefix}link_5"/>
       <axis xyz="0 1 0"/>
-      <limit lower="${radians(-115)}" upper="${radians(140)}" effort="29.0" velocity="${radians(475)}" />
+      <limit lower="${radians(-115)}" upper="${radians(140)}" effort="29.0" velocity="${radians(350)}" />
       <dynamics damping="0.0" friction="0.0"/>
     </joint>
@@ -207,5 +207,5 @@
       <child link="${prefix}link_6"/>
       <axis xyz="0 0 1"/>
-      <limit lower="${radians(-270)}" upper="${radians(270)}" effort="11.0" velocity="${radians(760)}" />
+      <limit lower="${radians(-270)}" upper="${radians(270)}" effort="11.0" velocity="${radians(600)}" />
       <dynamics damping="0.0" friction="0.0"/>
     </joint>

File: staubli_tx90_support/urdf/tx90xl_macro.xacro (robot description, xacro)
@@ -167,5 +167,5 @@
       (1) effort limit = 318 Nm if floor mounted
       (2) effort limit = 111 Nm if wall mounted -->
-      <limit lower="${radians(-180)}" upper="${radians(180)}" effort="318.0" velocity="${radians(400)}" />
+      <limit lower="${radians(-180)}" upper="${radians(180)}" effort="318.0" velocity="${radians(190)}" />
       <dynamics damping="0.0" friction="0.0"/>
     </joint>
@@ -175,5 +175,5 @@
       <child link="${prefix}link_2"/>
       <axis xyz="0 1 0"/>
-      <limit lower="${radians(-130)}" upper="${radians(147.5)}" effort="90.0" velocity="${radians(350)}" />
+      <limit lower="${radians(-130)}" upper="${radians(147.5)}" effort="90.0" velocity="${radians(160)}" />
       <dynamics damping="0.0" friction="0.0"/>
     </joint>
@@ -183,5 +183,5 @@
       <child link="${prefix}link_3"/>
       <axis xyz="0 1 0"/>
-      <limit lower="${radians(-145)}" upper="${radians(145)}" effort="53.0" velocity="${radians(410)}" />
+      <limit lower="${radians(-145)}" upper="${radians(145)}" effort="53.0" velocity="${radians(230)}" />
       <dynamics damping="0.0" friction="0.0"/>
     </joint>
@@ -191,5 +191,5 @@
       <child link="${prefix}link_4"/>
       <axis xyz="0 0 1"/>
-      <limit lower="${radians(-270)}" upper="${radians(270)}" effort="34.0" velocity="${radians(540)}" />
+      <limit lower="${radians(-270)}" upper="${radians(270)}" effort="34.0" velocity="${radians(400)}" />
       <dynamics damping="0.0" friction="0.0"/>
     </joint>
@@ -199,5 +199,5 @@
       <child link="${prefix}link_5"/>
       <axis xyz="0 1 0"/>
-      <limit lower="${radians(-115)}" upper="${radians(140)}" effort="29.0" velocity="${radians(475)}" />
+      <limit lower="${radians(-115)}" upper="${radians(140)}" effort="29.0" velocity="${radians(345)}" />
       <dynamics damping="0.0" friction="0.0"/>
     </joint>
@@ -207,5 +207,5 @@
       <child link="${prefix}link_6"/>
       <axis xyz="0 0 1"/>
-      <limit lower="${radians(-270)}" upper="${radians(270)}" effort="11.0" velocity="${radians(760)}" />
+      <limit lower="${radians(-270)}" upper="${radians(270)}" effort="11.0" velocity="${radians(600)}" />
       <dynamics damping="0.0" friction="0.0"/>
     </joint>
